Commit message: Update urdf model.

File: src/motor_control/urdf/inverted_pendulum.urdf (robot description, URDF)
Before this commit: robot motor_xacro, 2 links, 1 joints
Links:
- link pendulum: geometry collision cylinder length=${length_pendulum} radius=${radius_pendulum}; visual cylinder length=${length_pendulum} radius=${radius_pendulum}
Joints:
- removed joint None
- added joint motor_to_pendulum: type continuous, parent motor, child pendulum, origin xyz=0.16 0 0.03 rpy=-1.5707 0 0, axis 1 0 0

Commit message: Model is now in rviz visible.

File: src/motor_control/urdf/inverted_pendulum.urdf (robot description, URDF)
Before this commit: robot motor_xacro, 2 links, 1 joints
Links:
- link motor: mass None -> 0.8
- link pendulum: mass None -> 1.3565; geometry collision cylinder length=0.4 radius=0.02; visual cylinder length=0.4 radius=0.02
