Commit message: Update model of motor_stick.

File: src/motor_control/urdf/motor_stick.urdf (robot description, URDF)
Before this commit: robot motor_stick, 2 links, 1 joints
Links:
- added link stick; collision cylinder length=0.40 radius=0.03; visual cylinder length=0.40 radius=0.03

Commit message: Update model of motor_stick.

File: src/motor_control/urdf/motor_stick.urdf (robot description, URDF)
Before this commit: robot motor_stick, 3 links, 1 joints
Links:
- link motor: mass 1 -> 6; geometry collision box size=0.16 0.1 0.1; visual box size=0.16 0.1 0.1
- link stick: mass None -> 1.5; geometry collision cylinder length=0.40 radius=0.006; visual cylinder length=0.40 radius=0.006
Joints:
- added joint motor_to_stick: type revolute, parent motor, child stick, origin xyz=0 0 0.1 rpy=0 0 0, axis 0 1 0, limit lower=-1.5707 upper=1.5707 effort=10 velocity=5
